File: pcb/socotitoare/numpad.kicad_pcb (KiCad board)
At the start: 2 copper layers, 80 x 53 mm, 20 parts, among them J1 display, SW1 SW_Push, SW10 RotaryEncoder_Switch, SW2 SW_Push, SW3 SW_Push, SW4 SW_Push, U1 XIAO-RP2040-DIP

Commit message: v2
Parts:
- removed J1: display, SSD1306:SSD1306-0.91-OLED-4pin-128x32
- added U2: OLED_0.91_128x32, Hackclub Footprints:OLED_0.91_128x32, F.Cu at (167.9, 70.8)
- D1, D2, D3, D4, D5: value SK6812MINI -> SK6812MINI-E; footprint LED_SMD:LED_SK6812MINI_PLCC4_3.5x3.5mm_P1.75mm -> Hackclub Footprints:MX_SK6812MINI-E_REV
- moved D5 5.10 mm to (180.5, 81.3)
- moved D3 5.09 mm to (161.3, 110.5)
- moved D1 5.09 mm to (123.6, 110.5)
- moved D2 5.09 mm to (142.7, 110.5)
- moved D4 5.09 mm to (180.8, 110.5)
- moved REF** 2.50 mm to (186.9, 111.9)
- moved REF** 2.50 mm to (117.1, 111.9)
Connections:
- D1 pad 1: Net-(D1-DOUT) -> VCC
- D1 pad 2: GND -> Net-(D1-DOUT)
- D1 pad 3: SK6812 -> GND
- D1 pad 4: VCC -> SK6812
- D2 pad 1: Net-(D2-DOUT) -> VCC
- D2 pad 2: GND -> Net-(D2-DOUT)
- D2 pad 3: Net-(D1-DOUT) -> GND
- D2 pad 4: VCC -> Net-(D1-DOUT)
- D3 pad 1: Net-(D3-DOUT) -> VCC
- D3 pad 2: GND -> Net-(D3-DOUT)
- D3 pad 3: Net-(D2-DOUT) -> GND
- D3 pad 4: VCC -> Net-(D2-DOUT)
- D4 pad 1: Net-(D4-DOUT) -> VCC
- D4 pad 2: GND -> Net-(D4-DOUT)
- D4 pad 3: Net-(D3-DOUT) -> GND
- D4 pad 4: VCC -> Net-(D3-DOUT)
- D5 pad 1: unconnected-(D5-DOUT-Pad1) -> VCC
- D5 pad 2: GND -> unconnected-(D5-DOUT-Pad2)
- D5 pad 3: Net-(D4-DOUT) -> GND
- D5 pad 4: VCC -> Net-(D4-DOUT)
Routing:
- net Net-(D2-DOUT): track 23.3 -> 14.0 mm
- net Net-(D1-DOUT): track 23.3 -> 14.5 mm
- net Net-(D3-DOUT): track 23.3 -> 14.9 mm
- net VCC: track 176.7 -> 184.1 mm, vias 0 -> 2
- net GND: track 196.6 -> 191.2 mm
- net SK6812: track 72.8 -> 67.9 mm, vias 0 -> 1
- net Net-(D4-DOUT): track 38.4 -> 43.2 mm, vias 2 -> 0
