File: pcb/socotitoare/numpad.kicad_sch (KiCad schematic)
At the start: 17 parts, among them J1 Conn_01x04, SW1 SW_Push, SW10 RotaryEncoder_Switch, SW2 SW_Push, SW3 SW_Push, SW4 SW_Push, U1 XIAO-RP2040-DIP

Commit message: v2
Parts:
- removed D1, D2, D3, D4, D5: SK6812MINI, LED_SMD:LED_SK6812MINI_PLCC4_3.5x3.5mm_P1.75mm, symbol LED:SK6812MINI
- removed J1: Conn_01x04, SSD1306:SSD1306-0.91-OLED-4pin-128x32, symbol Connector_Generic:Conn_01x04
- added D1, D2, D3, D4, D5: SK6812MINI-E, Hackclub Footprints:MX_SK6812MINI-E_REV, symbol Hackclub Symbols:SK6812MINI-E
- added U2: OLED_0.91_128x32, Hackclub Footprints:OLED_0.91_128x32, symbol Hackclub Symbols:OLED_0.91_128x32
Connections:
- net GND: now also D1.3 (VSS), D2.3 (VSS), D3.3 (VSS), D4.3 (VSS), D5.3 (VSS), U2.1 (GND)
- net SCL: now also U2.3 (SCL)
- net SDA: now also U2.4 (SDA)
- net SK6812: now also D1.4 (DIN)
- net VCC: now also D1.1 (VDD), D2.1 (VDD), D3.1 (VDD), D4.1 (VDD), D5.1 (VDD), U2.2 (VCC)
- new net: D1.2 (DOUT), D2.4 (DIN)
- new net: D4.2 (DOUT), D5.4 (DIN)
- new net: D3.2 (DOUT), D4.4 (DIN)
- new net: D2.2 (DOUT), D3.4 (DIN)
